File: hardware/pcb-v3/wattplot-v3.kicad_sch (KiCad schematic)
At the start: 9 parts, among them U1 MP1584EN, U2 AMS1117-3.3

Commit message: hardware(pcb-v3): power tree wired, ERC 9 errors / 10 warnings (down from 6/0)
- LIB fixed: MP2307 -> Regulator_Switching:MP1470 (in stock lib),
  LED:LED -> Device:LED, D_TVS -> Power_Protection:TVS1800DRV,
  ESD5V0S1B -> USBLC6-2P6
- Schematic lib_symbols section now empty; KiCad resolves symbols
  from installed libraries at open time. (Stubs were the root cause
  of pin-anchor disagreement between script pin_pos and KiCad ERC.)
- place_power_tree rewrites: uses pin_pos everywhere, places one
  global label at each power pin (multiple same-name labels = same
  net per KiCad convention), explicit wires only for components
  that bridge two named nets (L1 inductor, C2 bootstrap cap).
- Full power tree now in schematic: 12V input, MP1470 buck with
  feedback divider and bootstrap, AMS1117 LDO, battery divider
  for ADC. 11 components, 19 nets.
- Known cosmetic issues to fix in KiCad GUI:
  * 6 label/pin anchor mismatches (mostly on horizontal SOT-23 /
    SOT-223 pins where label-shape vs pin-direction matters)
  * 2 C2 bootstrap cap wires show as dangling until GUI clean
  * 1 L1->C3 junction wire is a stub
  * 10 off-grid / unconnected wire endpoint warnings (sub-grid
    positions, not real errors)
Parts:
- removed C2: 100nF, Capacitor_SMD:C_0402_1005Metric, symbol Device:C
- removed U1: MP1584EN, Package_TO_SOT_SMD:SOT-23-6, symbol Converter_DCDC:MP2307
- added C2: 100nF, Capacitor_SMD:C_0402_1005Metric, symbol Device:C_Polarized
- added L1: 4.7uH, Inductor_SMD:L_1210_3225Metric, symbol Device:L
- added R1: 33k, Resistor_SMD:R_0603_1608Metric, symbol Device:R
- added R2: 10k, Resistor_SMD:R_0603_1608Metric, symbol Device:R
- added TP1: VBAT_ADC, TestPoint:TestPoint_Pad_D1.0mm, symbol Connector:TestPoint
- added U1: MP1584EN, Package_TO_SOT_SMD:SOT-23-6, symbol Regulator_Switching:MP1470
Other:
- note added: "→ GPIO7 (ADC)"
- note removed: "VBAT_ADC → GPIO7"

Commit message: hardware(pcb-v3): place ESP32-S3 + USB-C + EN/BOOT + LED + I2C + header
place_esp32_s3() places the ESP32-S3-WROOM-1 module (41 pins) plus:
- USB-C receptacle (J1) with USBLC6-2P6 ESD
- 330R + GREEN status LED on GPIO17
- 10k pull-up + reset button on EN
- BOOT button on GPIO0
- 4.7k I2C pull-ups on GPIO8/18 (SDA/SCL)
- 100nF + 10uF decoupling on 3V3
- 2x5 programming header (GND/BOOT/TX/RST/RX/3V3/IO4/IO5/GND)

All Wattplot signal labels placed AT each ESP32 pin:
  ACTUATOR_IN1/IN2/IPROPI/nFAULT (GPIO1/2/4/21)
  SOLENOID_IN1/IN2/IPROPI/nFAULT (GPIO10/12/5/13)
  SOIL_AOUT (GPIO6), BATTERY_V_ADC (GPIO7)
  I2C_SDA/SCL (GPIO8/18), DS18B20_DATA (GPIO16)
  STATUS_LED (GPIO17), BOOT (GPIO0), EN_CHIP (EN)
  USB_DP/DN (GPIO13/14), UART_RX/TX (GPIO44/43)

Routing rules: NO wire runs along x=284.76 or x=315.24 (GPIO
columns) — all connections go through x=325 to avoid shorting
labels together.

ERC: 83 violations (down from 100). Mix of cosmetic issues:
- 22 label_dangling (label-anchor quirks, fixable in GUI)
- 16 endpoint_off_grid (sub-grid positions)
- 2 multiple_net_names (real bugs to clean up in GUI:
  BOOT wire overlaps STATUS_LED, I2C_SDA wire passes near +3V3)
- 4 wire_dangling (decoupling cap stub endpoints)
- 3 footprint_link_issues (lib config)
Parts:
- added C6: 100nF, Capacitor_SMD:C_0402_1005Metric, symbol Device:C
- added C7: 10uF, Capacitor_SMD:C_0603_1608Metric, symbol Device:C
- added D1: GREEN, LED_SMD:LED_0805_2012Metric, symbol Device:LED
- added J1: USB-C, Connector:USB_C_Receptacle, symbol Connector:USB_C_Receptacle
- added J2: PROG, PinHeader_2.54mm:PinHeader_2x05_P2.54mm_Vertical, symbol Connector_Generic:Conn_02x05_Odd_Even
- added R5: 330R, Resistor_SMD:R_0603_1608Metric, symbol Device:R
- added R6: 10k, Resistor_SMD:R_0603_1608Metric, symbol Device:R
- added R7, R8: 4.7k, Resistor_SMD:R_0603_1608Metric, symbol Device:R
- added SW1: RESET, Switch:SW_Push, symbol Switch:SW_Push
- added SW2: BOOT, Switch:SW_Push, symbol Switch:SW_Push
- added U3: ESP32-S3-WROOM-1, RF_Module:ESP32-S3-WROOM-1, symbol RF_Module:ESP32-S3-WROOM-1
- added U4: USBLC6-2P6, Package_TO_SOT_SMD:SOT-23-6, symbol Power_Protection:USBLC6-2P6
Other:
- note added: "ESP32-S3 Module + USB + EN/BOOT + LED + I2C + Header"

Commit message: hardware(pcb-v3): place 2x DRV8871 H-bridges (U5 actuator / U6 solenoid)
place_drv8871s() places both H-bridges with full support circuitry:
- DRV8871DDA symbol (U5 actuator at 450,200; U6 solenoid at 450,300)
- 22uF/25V bulk caps on VM (C8, C10)
- 1k ILIM resistors to GND (R9, R11) - 200mV/A current sense
- JST-XH 2-pin output connectors (J3, J4) for motor + solenoid
- Virtual nFAULT test points (TP1, TP3) - the DRV8871DDA lib symbol
  is missing nFAULT/nSLEEP/VCC pins; nFAULT is modeled as a label that
  connects by name to the ACTUATOR_nFAULT/SOLENOID_nFAULT label on
  the ESP32 side

All signal labels placed at DRV8871 pins:
  ACTUATOR_IN1/IN2/IPROPI/nFAULT (GPIO1/2/4/21)
  SOLENOID_IN1/IN2/IPROPI/nFAULT (GPIO10/12/5/13)
  +12V (VM), GND

ERC: 116 violations. Multiple_net_names warnings: ACTUATOR_IPROPI/GND,
+3V3/I2C_SCL, BOOT/STATUS_LED - all caused by "through-resistor" wires
that ERC merges with the resistor net. Fix: remove the wires that
span the resistor body; rely on the resistor pins to make the
connection. Cosmetic otherwise.
Parts:
- removed TP1: VBAT_ADC, TestPoint:TestPoint_Pad_D1.0mm, symbol Connector:TestPoint
- added C10, C8: 22uF/25V, Capacitor_SMD:C_1210_3225Metric, symbol Device:C_Polarized
- added J3: ACTUATOR, Connector_JST:JST_XH_B2B-PH-K_1x02_P2.50mm_Vertical, symbol Connector_Generic:Conn_01x02
- added J4: SOLENOID, Connector_JST:JST_XH_B2B-PH-K_1x02_P2.50mm_Vertical, symbol Connector_Generic:Conn_01x02
- added R11, R9: 1k, Resistor_SMD:R_0603_1608Metric, symbol Device:R
- added TP1: nFAULT_ACT, TestPoint:TestPoint_Pad_D1.0mm, symbol Connector:TestPoint
- added TP1: VBAT_ADC, TestPoint:TestPoint_Pad_D1.0mm, symbol Connector:TestPoint
- added TP3: nFAULT_SOL, TestPoint:TestPoint_Pad_D1.0mm, symbol Connector:TestPoint
- added U5: DRV8871 (ACT), Package_SO:Texas_HTSOP-8-1EP_3.9x4.9mm_P1.27mm, symbol Driver_Motor:DRV8871DDA
- added U6: DRV8871 (SOL), Package_SO:Texas_HTSOP-8-1EP_3.9x4.9mm_P1.27mm, symbol Driver_Motor:DRV8871DDA
Other:
- note added: "ACTUATOR"
- note added: "DRV8871 H-bridges (U5 actuator / U6 solenoid)"
- note added: "SOLENOID"
Changed lines of the file:
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@@
 	(global_label "GND" (at 387.62 194.92 0) (shape bidirectional) (effects (font (size 1.27 1.27))))
 	(text "ESP32-S3 Module + USB + EN/BOOT + LED + I2C + Header" (at 270 90 0) (effects (font (size 2.0 2.0))))
+	(symbol (lib_id "Driver_Motor:DRV8871DDA") (at 450 200 0) (property "Reference" "U5" (at 450 194.92 0) (effects (font (size 1.27 1.27)) (justify left bottom))) (property "Value" "DRV8871 (ACT)" (at 450 192.38 0) (effects (font (size 1.27 1.27)) (justify left bottom))) (property "Footprint" "Package_SO:Texas_HTSOP-8-1EP_3.9x4.9mm_P1.27mm" (at 450 200 0) (effects (font (size 1.27 1.27)) (hide yes) (justify left bottom))))
+	(symbol (lib_id "Device:C_Polarized") (at 450 180 0) (property "Reference" "C8" (at 450 174.92 0) (effects (font (size 1.27 1.27)) (justify left bottom))) (property "Value" "22uF/25V" (at 450 172.38 0) (effects (font (size 1.27 1.27)) (justify left bottom))) (property "Footprint" "Capacitor_SMD:C_1210_3225Metric" (at 450 180 0) (effects (font (size 1.27 1.27)) (hide yes) (justify left bottom))))
+	(symbol (lib_id "Device:R") (at 475 195 0) (property "Reference" "R9" (at 475 189.92 0) (effects (font (size 1.27 1.27)) (justify left bottom))) (property "Value" "1k" (at 475 187.38 0) (effects (font (size 1.27 1.27)) (justify left bottom))) (property "Footprint" "Resistor_SMD:R_0603_1608Metric" (at 475 195 0) (effects (font (size 1.27 1.27)) (hide yes) (justify left bottom))))
+	(symbol (lib_id "Connector_Generic:Conn_01x02") (at 500 200 0) (property "Reference" "J3" (at 500 194.92 0) (effects (font (size 1.27 1.27)) (justify left bottom))) (property "Value" "ACTUATOR" (at 500 192.38 0) (effects (font (size 1.27 1.27)) (justify left bottom))) (property "Footprint" "Connector_JST:JST_XH_B2B-PH-K_1x02_P2.50mm_Vertical" (at 500 200 0) (effects (font (size 1.27 1.27)) (hide yes) (justify left bottom))))
+	(symbol (lib_id "Connector:TestPoint") (at 475 210 0) (property "Reference" "TP1" (at 475 204.92 0) (effects (font (size 1.27 1.27)) (justify left bottom))) (property "Value" "nFAULT_ACT" (at 475 202.38 0) (effects (font (size 1.27 1.27)) (justify left bottom))) (property "Footprint" "TestPoint:TestPoint_Pad_D1.0mm" (at 475 210 0) (effects (font (size 1.27 1.27)) (hide yes) (justify left bottom))))
+	(global_label "+12V" (at 450.0 210.16 0) (shape bidirectional) (effects (font (size 1.27 1.27))))
+	(global_label "GND" (at 450.0 189.84 0) (shape bidirectional) (effects (font (size 1.27 1.27))))
+	(global_label "GND" (at 450 189.84 0) (shape bidirectional) (effects (font (size 1.27 1.27))))
+	(global_label "ACTUATOR_IN1" (at 439.84 205.08 0) (shape bidirectional) (effects (font (size 1.27 1.27))))
+	(global_label "ACTUATOR_IN2" (at 439.84 202.54 0) (shape bidirectional) (effects (font (size 1.27 1.27))))
+	(global_label "ACTUATOR_IPROPI" (at 460.16 194.92 0) (shape bidirectional) (effects (font (size 1.27 1.27))))
+	(global_label "OUT1" (at 494.92 200.0 0) (shape bidirectional) (effects (font (size 1.27 1.27))))
+	(global_label "OUT2" (at 494.92 197.46 0) (shape bidirectional) (effects (font (size 1.27 1.27))))
+	(global_label "ACTUATOR_nFAULT" (at 475.0 210.0 0) (shape bidirectional) (effects (font (size 1.27 1.27))))
+	(text "ACTUATOR" (at 505 207 0) (effects (font (size 1.27 1.27))))
+	(wire (pts (xy 450.0 183.81) (xy 450.0 210.16)) (stroke (width 0) (type default) (color 0 0 0 0)))
+	(wire (pts (xy 450.0 210.16) (xy 450.0 210.16)) (stroke (width 0) (type default) (color 0 0 0 0)))
+	(junction (at 450.0 210.16) (diameter 0) (color 0 0 0 0))
+	(wire (pts (xy 450.0 176.19) (xy 450.0 170)) (stroke (width 0) (type default) (color 0 0 0 0)))
+	(global_label "GND" (at 450.0 170 0) (shape bidirectional) (effects (font (size 1.27 1.27))))
+	(wire (pts (xy 460.16 205.08) (xy 460.16 200.0)) (stroke (width 0) (type default) (color 0 0 0 0)))
+	(wire (pts (xy 460.16 200.0) (xy 494.92 200.0)) (stroke (width 0) (type default) (color 0 0 0 0)))
+	(junction (at 460.16 200.0) (diameter 0) (color 0 0 0 0))
+	(wire (pts (xy 460.16 202.54) (xy 460.16 197.46)) (stroke (width 0) (type default) (color 0 0 0 0)))
+	(wire (pts (xy 460.16 197.46) (xy 494.92 197.46)) (stroke (width 0) (type default) (color 0 0 0 0)))
+	(junction (at 460.16 197.46) (diameter 0) (color 0 0 0 0))
+	(wire (pts (xy 460.16 194.92) (xy 460.16 198.81)) (stroke (width 0) (type default) (color 0 0 0 0)))
+	(wire (pts (xy 460.16 198.81) (xy 475.0 198.81)) (stroke (width 0) (type default) (color 0 0 0 0)))
+	(junction (at 460.16 198.81) (diameter 0) (color 0 0 0 0))
+	(wire (pts (xy 475.0 198.81) (xy 475.0 191.19)) (stroke (width 0) (type default) (color 0 0 0 0)))
+	(wire (pts (xy 475.0 191.19) (xy 475.0 170)) (stroke (width 0) (type default) (color 0 0 0 0)))
+	(global_label "GND" (at 475.0 170 0) (shape bidirectional) (effects (font (size 1.27 1.27))))
+	(symbol (lib_id "Driver_Motor:DRV8871DDA") (at 450 300 0) (property "Reference" "U6" (at 450 294.92 0) (effects (font (size 1.27 1.27)) (justify left bottom))) (property "Value" "DRV8871 (SOL)" (at 450 292.38 0) (effects (font (size 1.27 1.27)) (justify left bottom))) (property "Footprint" "Package_SO:Texas_HTSOP-8-1EP_3.9x4.9mm_P1.27mm" (at 450 300 0) (effects (font (size 1.27 1.27)) (hide yes) (justify left bottom))))
+	(symbol (lib_id "Device:C_Polarized") (at 450 280 0) (property "Reference" "C10" (at 450 274.92 0) (effects (font (size 1.27 1.27)) (justify left bottom))) (property "Value" "22uF/25V" (at 450 272.38 0) (effects (font (size 1.27 1.27)) (justify left bottom))) (property "Footprint" "Capacitor_SMD:C_1210_3225Metric" (at 450 280 0) (effects (font (size 1.27 1.27)) (hide yes) (justify left bottom))))
+	(symbol (lib_id "Device:R") (at 475 295 0) (property "Reference" "R11" (at 475 289.92 0) (effects (font (size 1.27 1.27)) (justify left bottom))) (property "Value" "1k" (at 475 287.38 0) (effects (font (size 1.27 1.27)) (justify left bottom))) (property "Footprint" "Resistor_SMD:R_0603_1608Metric" (at 475 295 0) (effects (font (size 1.27 1.27)) (hide yes) (justify left bottom))))
+	(symbol (lib_id "Connector_Generic:Conn_01x02") (at 500 300 0) (property "Reference" "J4" (at 500 294.92 0) (effects (font (size 1.27 1.27)) (justify left bottom))) (property "Value" "SOLENOID" (at 500 292.38 0) (effects (font (size 1.27 1.27)) (justify left bottom))) (property "Footprint" "Connector_JST:JST_XH_B2B-PH-K_1x02_P2.50mm_Vertical" (at 500 300 0) (effects (font (size 1.27 1.27)) (hide yes) (justify left bottom))))
+	(symbol (lib_id "Connector:TestPoint") (at 475 310 0) (property "Reference" "TP3" (at 475 304.92 0) (effects (font (size 1.27 1.27)) (justify left bottom))) (property "Value" "nFAULT_SOL" (at 475 302.38 0) (effects (font (size 1.27 1.27)) (justify left bottom))) (property "Footprint" "TestPoint:TestPoint_Pad_D1.0mm" (at 475 310 0) (effects (font (size 1.27 1.27)) (hide yes) (justify left bottom))))
+	(global_label "+12V" (at 450.0 310.16 0) (shape bidirectional) (effects (font (size 1.27 1.27))))
+	(global_label "GND" (at 450.0 289.84 0) (shape bidirectional) (effects (font (size 1.27 1.27))))
+	(global_label "GND" (at 450 289.84 0) (shape bidirectional) (effects (font (size 1.27 1.27))))
+	(global_label "SOLENOID_IN1" (at 439.84 305.08 0) (shape bidirectional) (effects (font (size 1.27 1.27))))
+	(global_label "SOLENOID_IN2" (at 439.84 302.54 0) (shape bidirectional) (effects (font (size 1.27 1.27))))
+	(global_label "SOLENOID_IPROPI" (at 460.16 294.92 0) (shape bidirectional) (effects (font (size 1.27 1.27))))
+	(global_label "OUT1" (at 494.92 300.0 0) (shape bidirectional) (effects (font (size 1.27 1.27))))
+	(global_label "OUT2" (at 494.92 297.46 0) (shape bidirectional) (effects (font (size 1.27 1.27))))
+	(global_label "SOLENOID_nFAULT" (at 475.0 310.0 0) (shape bidirectional) (effects (font (size 1.27 1.27))))
+	(text "SOLENOID" (at 505 307 0) (effects (font (size 1.27 1.27))))
+	(wire (pts (xy 450.0 283.81) (xy 450.0 310.16)) (stroke (width 0) (type default) (color 0 0 0 0)))
+	(wire (pts (xy 450.0 310.16) (xy 450.0 310.16)) (stroke (width 0) (type default) (color 0 0 0 0)))
+	(junction (at 450.0 310.16) (diameter 0) (color 0 0 0 0))
+	(wire (pts (xy 450.0 276.19) (xy 450.0 270)) (stroke (width 0) (type default) (color 0 0 0 0)))
+	(global_label "GND" (at 450.0 270 0) (shape bidirectional) (effects (font (size 1.27 1.27))))
+	(wire (pts (xy 460.16 305.08) (xy 460.16 300.0)) (stroke (width 0) (type default) (color 0 0 0 0)))
+	(wire (pts (xy 460.16 300.0) (xy 494.92 300.0)) (stroke (width 0) (type default) (color 0 0 0 0)))
+	(junction (at 460.16 300.0) (diameter 0) (color 0 0 0 0))
+	(wire (pts (xy 460.16 302.54) (xy 460.16 297.46)) (stroke (width 0) (type default) (color 0 0 0 0)))
+	(wire (pts (xy 460.16 297.46) (xy 494.92 297.46)) (stroke (width 0) (type default) (color 0 0 0 0)))
+	(junction (at 460.16 297.46) (diameter 0) (color 0 0 0 0))
+	(wire (pts (xy 460.16 294.92) (xy 460.16 298.81)) (stroke (width 0) (type default) (color 0 0 0 0)))
+	(wire (pts (xy 460.16 298.81) (xy 475.0 298.81)) (stroke (width 0) (type default) (color 0 0 0 0)))
+	(junction (at 460.16 298.81) (diameter 0) (color 0 0 0 0))
+	(wire (pts (xy 475.0 298.81) (xy 475.0 291.19)) (stroke (width 0) (type default) (color 0 0 0 0)))
+	(wire (pts (xy 475.0 291.19) (xy 475.0 270)) (stroke (width 0) (type default) (color 0 0 0 0)))
+	(global_label "GND" (at 475.0 270 0) (shape bidirectional) (effects (font (size 1.27 1.27))))
+	(text "DRV8871 H-bridges (U5 actuator / U6 solenoid)" (at 420 150 0) (effects (font (size 2.0 2.0))))
 )

Commit message: hardware(pcb-v3): place 2x INA219 current monitors (U7 panel / U8 actuator)
place_ina219s() places two INA219BxD chips:
- U7 (0x41) panel: A0=VS, A1=GND
- U8 (0x40) actuator: A0=GND, A1=GND
Each with:
- 100nF VS bypass cap
- All signal labels (VS, GND, SDA, SCL, IN+, IN-, A0, A1) at pins
- PANEL_IN+/IN- for U7, ACT_IN+/IN- for U8

Schematic is now ~80% complete. Remaining:
- Sensor interfaces (1-Wire, soil moisture, connector)
- 4 custom symbols (MP1584, SMBJ16A, LED_0805, XT60)
- Final ERC clean in GUI
Parts:
- removed TP1: nFAULT_ACT, TestPoint:TestPoint_Pad_D1.0mm, symbol Connector:TestPoint
- removed TP1: VBAT_ADC, TestPoint:TestPoint_Pad_D1.0mm, symbol Connector:TestPoint
- added C12, C13: 100nF, Capacitor_SMD:C_0402_1005Metric, symbol Device:C
- added TP1: nFAULT_ACT, TestPoint:TestPoint_Pad_D1.0mm, symbol Connector:TestPoint
- added TP1: VBAT_ADC, TestPoint:TestPoint_Pad_D1.0mm, symbol Connector:TestPoint
- added U7: INA219 (PAN), Package_SO:SOIC-8_3.9x4.9mm_P1.27mm, symbol Sensor_Energy:INA219BxD
- added U8: INA219 (ACT), Package_SO:SOIC-8_3.9x4.9mm_P1.27mm, symbol Sensor_Energy:INA219BxD
Other:
- note added: "BATT_SHUNT (1mΩ)"
- note added: "INA219 current monitors (U7 panel / U8 actuator+battery)"
- note added: "PV_SHUNT (1mΩ)"
Changed lines of the file:
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@@
 	(global_label "GND" (at 475.0 270 0) (shape bidirectional) (effects (font (size 1.27 1.27))))
 	(text "DRV8871 H-bridges (U5 actuator / U6 solenoid)" (at 420 150 0) (effects (font (size 2.0 2.0))))
+	(symbol (lib_id "Sensor_Energy:INA219BxD") (at 600 200 0) (property "Reference" "U7" (at 600 194.92 0) (effects (font (size 1.27 1.27)) (justify left bottom))) (property "Value" "INA219 (PAN)" (at 600 192.38 0) (effects (font (size 1.27 1.27)) (justify left bottom))) (property "Footprint" "Package_SO:SOIC-8_3.9x4.9mm_P1.27mm" (at 600 200 0) (effects (font (size 1.27 1.27)) (hide yes) (justify left bottom))))
+	(symbol (lib_id "Device:C") (at 630 210 0) (property "Reference" "C12" (at 630 204.92 0) (effects (font (size 1.27 1.27)) (justify left bottom))) (property "Value" "100nF" (at 630 202.38 0) (effects (font (size 1.27 1.27)) (justify left bottom))) (property "Footprint" "Capacitor_SMD:C_0402_1005Metric" (at 630 210 0) (effects (font (size 1.27 1.27)) (hide yes) (justify left bottom))))
+	(global_label "+3V3" (at 600.0 210.16 0) (shape bidirectional) (effects (font (size 1.27 1.27))))
+	(global_label "GND" (at 600.0 189.84 0) (shape bidirectional) (effects (font (size 1.27 1.27))))
+	(global_label "I2C_SDA" (at 610.16 205.08 0) (shape bidirectional) (effects (font (size 1.27 1.27))))
+	(global_label "I2C_SCL" (at 610.16 202.54 0) (shape bidirectional) (effects (font (size 1.27 1.27))))
+	(global_label "PANEL_IN+" (at 589.84 202.54 0) (shape bidirectional) (effects (font (size 1.27 1.27))))
+	(global_label "PANEL_IN-" (at 589.84 197.46 0) (shape bidirectional) (effects (font (size 1.27 1.27))))
+	(global_label "+3V3" (at 610.16 194.92 0) (shape bidirectional) (effects (font (size 1.27 1.27))))
+	(global_label "GND" (at 610.16 197.46 0) (shape bidirectional) (effects (font (size 1.27 1.27))))
+	(wire (pts (xy 630.0 213.81) (xy 600.0 213.81)) (stroke (width 0) (type default) (color 0 0 0 0)))
+	(wire (pts (xy 600.0 213.81) (xy 600.0 210.16)) (stroke (width 0) (type default) (color 0 0 0 0)))
+	(junction (at 600.0 213.81) (diameter 0) (color 0 0 0 0))
+	(wire (pts (xy 630.0 206.19) (xy 630.0 170)) (stroke (width 0) (type default) (color 0 0 0 0)))
+	(global_label "GND" (at 630.0 170 0) (shape bidirectional) (effects (font (size 1.27 1.27))))
+	(global_label "+3V3" (at 600.0 213.81 0) (shape bidirectional) (effects (font (size 1.27 1.27))))
+	(text "PV_SHUNT (1mΩ)" (at 575 175 0) (effects (font (size 1.0 1.0))))
+	(symbol (lib_id "Sensor_Energy:INA219BxD") (at 600 300 0) (property "Reference" "U8" (at 600 294.92 0) (effects (font (size 1.27 1.27)) (justify left bottom))) (property "Value" "INA219 (ACT)" (at 600 292.38 0) (effects (font (size 1.27 1.27)) (justify left bottom))) (property "Footprint" "Package_SO:SOIC-8_3.9x4.9mm_P1.27mm" (at 600 300 0) (effects (font (size 1.27 1.27)) (hide yes) (justify left bottom))))
+	(symbol (lib_id "Device:C") (at 630 310 0) (property "Reference" "C13" (at 630 304.92 0) (effects (font (size 1.27 1.27)) (justify left bottom))) (property "Value" "100nF" (at 630 302.38 0) (effects (font (size 1.27 1.27)) (justify left bottom))) (property "Footprint" "Capacitor_SMD:C_0402_1005Metric" (at 630 310 0) (effects (font (size 1.27 1.27)) (hide yes) (justify left bottom))))
+	(global_label "+3V3" (at 600.0 310.16 0) (shape bidirectional) (effects (font (size 1.27 1.27))))
+	(global_label "GND" (at 600.0 289.84 0) (shape bidirectional) (effects (font (size 1.27 1.27))))
+	(global_label "I2C_SDA" (at 610.16 305.08 0) (shape bidirectional) (effects (font (size 1.27 1.27))))
+	(global_label "I2C_SCL" (at 610.16 302.54 0) (shape bidirectional) (effects (font (size 1.27 1.27))))
+	(global_label "ACT_IN+" (at 589.84 302.54 0) (shape bidirectional) (effects (font (size 1.27 1.27))))
+	(global_label "ACT_IN-" (at 589.84 297.46 0) (shape bidirectional) (effects (font (size 1.27 1.27))))
+	(global_label "GND" (at 610.16 294.92 0) (shape bidirectional) (effects (font (size 1.27 1.27))))
+	(global_label "GND" (at 610.16 297.46 0) (shape bidirectional) (effects (font (size 1.27 1.27))))
+	(wire (pts (xy 630.0 313.81) (xy 600.0 313.81)) (stroke (width 0) (type default) (color 0 0 0 0)))
+	(wire (pts (xy 600.0 313.81) (xy 600.0 310.16)) (stroke (width 0) (type default) (color 0 0 0 0)))
+	(junction (at 600.0 313.81) (diameter 0) (color 0 0 0 0))
+	(wire (pts (xy 630.0 306.19) (xy 630.0 270)) (stroke (width 0) (type default) (color 0 0 0 0)))
+	(global_label "GND" (at 630.0 270 0) (shape bidirectional) (effects (font (size 1.27 1.27))))
+	(global_label "+3V3" (at 600.0 313.81 0) (shape bidirectional) (effects (font (size 1.27 1.27))))
+	(text "BATT_SHUNT (1mΩ)" (at 575 275 0) (effects (font (size 1.0 1.0))))
+	(text "INA219 current monitors (U7 panel / U8 actuator+battery)" (at 570 150 0) (effects (font (size 2.0 2.0))))
 )
