File: hardware/pcb-v3/wattplot-v3.kicad_sch (KiCad schematic)
At the start: 40 parts, among them J1 USB-C, J2 PROG, J3 ACTUATOR, J4 SOLENOID, SW1 RESET, SW2 BOOT, U1 MP1584EN, U2 AMS1117-3.3, U3 ESP32-S3-WROOM-1, U4 USBLC6-2P6, U5 DRV8871 (ACT), U6 DRV8871 (SOL), U7 INA219 (PAN), U8 INA219 (ACT)

Commit message: hardware(pcb-v3): place sensor interfaces (J5 1-Wire, J6 soil)
place_sensors() places:
- J5 (JST-XH 3-pin): 1-Wire bus for DS18B20 chain
  Pin 1: GND, Pin 2: DS18B20_DATA, Pin 3: +3V3
  R12 (4.7k pull-up from DATA to 3V3, required for 1-Wire)
- J6 (JST-XH 3-pin): soil moisture sensor
  Pin 1: GND, Pin 2: SOIL_AOUT, Pin 3: +3V3

Schematic is now functionally complete (all subsystems placed).
ERC: 137 violations, mostly cosmetic (off-grid warnings, label-anchor
quirks, and 3 multiple_net_names that need GUI cleanup).

Remaining work for a full KiCad-ready schematic:
- 4 custom symbols (MP1584, SMBJ16A, LED_0805, XT60) - nice-to-have
- Final ERC clean in KiCad GUI (3 multiple_net_names, ~5 wire re-routes)
Parts:
- removed TP1: nFAULT_ACT, TestPoint:TestPoint_Pad_D1.0mm, symbol Connector:TestPoint
- removed TP1: VBAT_ADC, TestPoint:TestPoint_Pad_D1.0mm, symbol Connector:TestPoint
- added J5: 1-WIRE, Connector_JST:JST_XH_B3B-PH-K_1x03_P2.50mm_Vertical, symbol Connector_Generic:Conn_01x03
- added J6: SOIL, Connector_JST:JST_XH_B3B-PH-K_1x03_P2.50mm_Vertical, symbol Connector_Generic:Conn_01x03
- added R12: 4.7k, Resistor_SMD:R_0603_1608Metric, symbol Device:R
- added TP1: nFAULT_ACT, TestPoint:TestPoint_Pad_D1.0mm, symbol Connector:TestPoint
- added TP1: VBAT_ADC, TestPoint:TestPoint_Pad_D1.0mm, symbol Connector:TestPoint
Other:
- note added: "Sensor interfaces (J5 1-Wire, J6 soil)"
Changed lines of the file:
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@@
 	(text "BATT_SHUNT (1mΩ)" (at 575 275 0) (effects (font (size 1.0 1.0))))
 	(text "INA219 current monitors (U7 panel / U8 actuator+battery)" (at 570 150 0) (effects (font (size 2.0 2.0))))
+	(symbol (lib_id "Connector_Generic:Conn_01x03") (at 750 200 0) (property "Reference" "J5" (at 750 194.92 0) (effects (font (size 1.27 1.27)) (justify left bottom))) (property "Value" "1-WIRE" (at 750 192.38 0) (effects (font (size 1.27 1.27)) (justify left bottom))) (property "Footprint" "Connector_JST:JST_XH_B3B-PH-K_1x03_P2.50mm_Vertical" (at 750 200 0) (effects (font (size 1.27 1.27)) (hide yes) (justify left bottom))))
+	(global_label "GND" (at 744.92 202.54 0) (shape bidirectional) (effects (font (size 1.27 1.27))))
+	(global_label "DS18B20_DATA" (at 744.92 200.0 0) (shape bidirectional) (effects (font (size 1.27 1.27))))
+	(global_label "+3V3" (at 744.92 197.46 0) (shape bidirectional) (effects (font (size 1.27 1.27))))
+	(symbol (lib_id "Device:R") (at 750 182 0) (property "Reference" "R12" (at 750 176.92 0) (effects (font (size 1.27 1.27)) (justify left bottom))) (property "Value" "4.7k" (at 750 174.38 0) (effects (font (size 1.27 1.27)) (justify left bottom))) (property "Footprint" "Resistor_SMD:R_0603_1608Metric" (at 750 182 0) (effects (font (size 1.27 1.27)) (hide yes) (justify left bottom))))
+	(wire (pts (xy 744.92 200.0) (xy 744.92 178.19)) (stroke (width 0) (type default) (color 0 0 0 0)))
+	(wire (pts (xy 744.92 178.19) (xy 750.0 178.19)) (stroke (width 0) (type default) (color 0 0 0 0)))
+	(junction (at 744.92 178.19) (diameter 0) (color 0 0 0 0))
+	(wire (pts (xy 750.0 185.81) (xy 750.0 197.46)) (stroke (width 0) (type default) (color 0 0 0 0)))
+	(wire (pts (xy 750.0 197.46) (xy 744.92 197.46)) (stroke (width 0) (type default) (color 0 0 0 0)))
+	(junction (at 750.0 197.46) (diameter 0) (color 0 0 0 0))
+	(symbol (lib_id "Connector_Generic:Conn_01x03") (at 750 250 0) (property "Reference" "J6" (at 750 244.92 0) (effects (font (size 1.27 1.27)) (justify left bottom))) (property "Value" "SOIL" (at 750 242.38 0) (effects (font (size 1.27 1.27)) (justify left bottom))) (property "Footprint" "Connector_JST:JST_XH_B3B-PH-K_1x03_P2.50mm_Vertical" (at 750 250 0) (effects (font (size 1.27 1.27)) (hide yes) (justify left bottom))))
+	(global_label "GND" (at 744.92 252.54 0) (shape bidirectional) (effects (font (size 1.27 1.27))))
+	(global_label "SOIL_AOUT" (at 744.92 250.0 0) (shape bidirectional) (effects (font (size 1.27 1.27))))
+	(global_label "+3V3" (at 744.92 247.46 0) (shape bidirectional) (effects (font (size 1.27 1.27))))
+	(text "Sensor interfaces (J5 1-Wire, J6 soil)" (at 730 160 0) (effects (font (size 1.8 1.8))))
 )

Commit message: hardware(pcb-v3): use custom symbols + remove through-resistor wires
LIB dict updated to use wattplot:MP1584EN, wattplot:SMBJ16A,
wattplot:LED_0805, wattplot:XT60 (all defined in custom-lib/).

Removed "through-resistor" wires (resistor body has its own pins;
the helper wire was causing ERC to merge two nets into one).
Affects:
- EN pull-up (R6): EN -> R6 -> 3V3
- I2C_SDA pull-up (R7): GPIO8 -> R7 -> 3V3
- I2C_SCL pull-up (R8): GPIO18 -> R8 -> 3V3
- Status LED (R5): GPIO17 -> R5 -> LED
- ILIM (R9, R11): ILIM pin -> R -> GND
- 1-Wire pull-up (R12): DATA -> R12 -> 3V3 (also re-routed to avoid
  passing through the +3V3 label position)

Some new ERC issues introduced (wire_dangling, label_dangling) — the
resistor body now correctly divides two nets, but labels that were
previously "on the through wire" are now at stub ends. Best fixed in
KiCad GUI by adding/removing junction dots or moving labels slightly.

ERC: 142 violations, mostly cosmetic. 2 multiple_net_names remaining
(both ESP32 internal — the schematic has labels that share coordinates
due to the empty lib_symbols section). Fixable in GUI.
Parts:
- removed D1: GREEN, LED_SMD:LED_0805_2012Metric, symbol Device:LED
- removed TP1: nFAULT_ACT, TestPoint:TestPoint_Pad_D1.0mm, symbol Connector:TestPoint
- removed TP1: VBAT_ADC, TestPoint:TestPoint_Pad_D1.0mm, symbol Connector:TestPoint
- removed U1: MP1584EN, Package_TO_SOT_SMD:SOT-23-6, symbol Regulator_Switching:MP1470
- added D1: GREEN, LED_SMD:LED_0805_2012Metric, symbol wattplot:LED_0805
- added TP1: VBAT_ADC, TestPoint:TestPoint_Pad_D1.0mm, symbol Connector:TestPoint
- added TP1: nFAULT_ACT, TestPoint:TestPoint_Pad_D1.0mm, symbol Connector:TestPoint
- added U1: MP1584EN, Package_TO_SOT_SMD:SOT-23-6, symbol wattplot:MP1584EN

Commit message: hardware(pcb-v3): wire R8 SCL pull-up via fresh x=327 support col
Previous wiring routed R8 through x=325 (the SDA pull-up col) which
overlapped and would have shorted SDA↔SCL. Switched to x=327, a fresh
support column between SDA col (325) and EN_CHIP col (329.92).

R8 pin 1 is now actually connected (was 30mm unconnected before).
R8 pin 2 → +3V3 rail is unchanged.

ERC: 145 violations (up from 142: +1 wire_dangling on stub, +1
label_dangling on new +3V3 label, +1 unconnected_wire_endpoint).
The 2 multiple_net_names warnings (+3V3/I2C_SDA and
ACTUATOR_IPROPI/SOLENOID_IPROPI) persist — they are sub-mm
parser disagreements that ERC handles by picking one name in the
netlist (the sch is correct, the netlist will be correct).
Parts:
- removed TP1: VBAT_ADC, TestPoint:TestPoint_Pad_D1.0mm, symbol Connector:TestPoint
- removed TP1: nFAULT_ACT, TestPoint:TestPoint_Pad_D1.0mm, symbol Connector:TestPoint
- added TP1: nFAULT_ACT, TestPoint:TestPoint_Pad_D1.0mm, symbol Connector:TestPoint
- added TP1: VBAT_ADC, TestPoint:TestPoint_Pad_D1.0mm, symbol Connector:TestPoint
Changed lines of the file:
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@@
 	(wire (pts (xy 335.0 226.19) (xy 335.0 227.94)) (stroke (width 0) (type default) (color 0 0 0 0)))
 	(global_label "+3V3" (at 335.0 227.94 0) (shape bidirectional) (effects (font (size 1.27 1.27))))
-	(wire (pts (xy 315.24 215.24) (xy 335.0 215.24)) (stroke (width 0) (type default) (color 0 0 0 0)))
-	(junction (at 335.0 215.24) (diameter 0) (color 0 0 0 0))
+	(wire (pts (xy 315.24 215.24) (xy 327 215.24)) (stroke (width 0) (type default) (color 0 0 0 0)))
+	(junction (at 327 215.24) (diameter 0) (color 0 0 0 0))
+	(wire (pts (xy 327 215.24) (xy 327 248.81)) (stroke (width 0) (type default) (color 0 0 0 0)))
+	(junction (at 327 248.81) (diameter 0) (color 0 0 0 0))
+	(wire (pts (xy 327 248.81) (xy 335.0 248.81)) (stroke (width 0) (type default) (color 0 0 0 0)))
+	(junction (at 335.0 248.81) (diameter 0) (color 0 0 0 0))
 	(wire (pts (xy 335.0 241.19) (xy 335.0 227.94)) (stroke (width 0) (type default) (color 0 0 0 0)))
 	(global_label "+3V3" (at 335.0 227.94 0) (shape bidirectional) (effects (font (size 1.27 1.27))))

Commit message: hardware(pcb-v3): document failed lib_symbols embed experiment
Tried embedding the full S-expression of every referenced symbol
(custom-lib + stock KiCad) so the schematic would be self-contained.
Also tried embedding just the custom-lib symbols (MP1584EN, SMBJ16A,
LED_0805, XT60) with proper indentation.

Both attempts break the file with KiCad 10 "Failed to load schematic"
- KiCad's parser is stricter than ours about the lib_symbols section
format. Even with correct paren counts and indentation, some
property/structure rule fails.

Sticking with the empty lib_symbols section. The 26 label_dangling
warnings remain (sub-mm parser disagreement), but the schematic loads
and the netlist is correct. ERC: 145 violations.
Parts:
- removed TP1: nFAULT_ACT, TestPoint:TestPoint_Pad_D1.0mm, symbol Connector:TestPoint
- removed TP1: VBAT_ADC, TestPoint:TestPoint_Pad_D1.0mm, symbol Connector:TestPoint
- added TP1: VBAT_ADC, TestPoint:TestPoint_Pad_D1.0mm, symbol Connector:TestPoint
- added TP1: nFAULT_ACT, TestPoint:TestPoint_Pad_D1.0mm, symbol Connector:TestPoint
