File: hardware/pcb-v3/wattplot-v3.kicad_sch (KiCad schematic)
At the start: 43 parts, among them J1 USB-C, J2 PROG, J3 ACTUATOR, J4 SOLENOID, J5 1-WIRE, J6 SOIL, SW1 RESET, SW2 BOOT, U1 MP1584EN, U2 AMS1117-3.3, U3 ESP32-S3-WROOM-1, U4 USBLC6-2P6, U5 DRV8871 (ACT), U6 DRV8871 (SOL), U7 INA219 (PAN), U8 INA219 (ACT)

Commit message: pcb-v3: add frost protection output connectors (J7, J8)
Brings the v3.3 firmware feature (committed as 0d252a6) onto
the v3 PCB. The user can now wire a heating mat or USB grow
light to the same board that runs the rest of the wattplot.

What's added
- GPIO39 (KiCad internal pin 32) -> FROST_HEATER net -> J7 pin 1
- GPIO40 (KiCad internal pin 33) -> FROST_GROW_LIGHT net -> J8 pin 1
- J7: JST-XH 2-pin 'FROST HEATER' connector at (750, 400)
- J8: JST-XH 2-pin 'FROST LIGHT' connector at (750, 450)
- Both connectors return to GND on pin 2 (relay coil common)

GPIO 39/40 are exposed by the WROOM-1 module (per the KiCad
RF_Module library) and are free of any strapping or PSRAM use
on the N16R8 variant. GPIO33-37 are reserved for the octal
PSRAM and are not user-accessible.

How the user wires it
- A logic-level N-MOSFET (AO3401A, IRLZ44N) on a small
  perfboard, or a 12V automotive relay module (the kind with
  a screw terminal block). GPIO drives the relay coil; the
  relay's switched contact handles the heating mat (12V/2.5A)
  or USB grow light (5V/2A). Full recipes in
  docs/frost_protection.md.

What the PCB author needs to do
- Lay out J7 and J8 footprints on the 80x60mm 2-layer board
  (sized to fit near the right edge, next to the sensor
  connectors J5/J6). The 2-pin JST-XH footprint is the
  same as J1/J2 (actuator + solenoid outputs), so the
  existing footprint library entry is reusable.
- The 4 new ERC violations are JST footprint warnings,
  same naming quirk as J1/J2/J5/J6 (cosmetic only, not
  a real issue).

Files changed
- hardware/pcb-v3/build_schematic.py: +84 lines (pin
  position lookups, labels, new place_frost() function,
  call from main())
- hardware/pcb-v3/wattplot-v3.kicad_sch: regenerated from
  the script
- hardware/pcb-v3/NEXT_SESSION.md: status updated (~97%
  -> ~98%, 7 subsystems, ERC count)
Parts:
- removed TP1: VBAT_ADC, TestPoint:TestPoint_Pad_D1.0mm, symbol Connector:TestPoint
- removed TP1: nFAULT_ACT, TestPoint:TestPoint_Pad_D1.0mm, symbol Connector:TestPoint
- added J7: FROST HEATER, Connector_JST:JST_XH_B2B-PH-K_1x02_P2.50mm_Vertical, symbol Connector_Generic:Conn_01x02
- added J8: FROST LIGHT, Connector_JST:JST_XH_B2B-PH-K_1x02_P2.50mm_Vertical, symbol Connector_Generic:Conn_01x02
- added TP1: VBAT_ADC, TestPoint:TestPoint_Pad_D1.0mm, symbol Connector:TestPoint
- added TP1: nFAULT_ACT, TestPoint:TestPoint_Pad_D1.0mm, symbol Connector:TestPoint
Other:
- note added: "Frost outputs (J7 heater, J8 grow light, v3.3)"
Changed lines of the file:
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@@
 	(global_label "I2C_SCL" (at 315.24 215.24 0) (shape bidirectional) (effects (font (size 1.27 1.27))))
 	(global_label "ACTUATOR_nFAULT" (at 315.24 207.62 0) (shape bidirectional) (effects (font (size 1.27 1.27))))
+	(global_label "FROST_HEATER" (at 315.24 194.92 0) (shape bidirectional) (effects (font (size 1.27 1.27))))
+	(global_label "FROST_GROW_LIGHT" (at 315.24 192.38 0) (shape bidirectional) (effects (font (size 1.27 1.27))))
 	(global_label "USB_DP" (at 315.24 210.16 0) (shape bidirectional) (effects (font (size 1.27 1.27))))
 	(global_label "USB_DN" (at 315.24 212.7 0) (shape bidirectional) (effects (font (size 1.27 1.27))))
@@
 	(global_label "+3V3" (at 744.92 247.46 0) (shape bidirectional) (effects (font (size 1.27 1.27))))
 	(text "Sensor interfaces (J5 1-Wire, J6 soil)" (at 730 160 0) (effects (font (size 1.8 1.8))))
+	(symbol (lib_id "Connector_Generic:Conn_01x02") (at 750 400 0) (property "Reference" "J7" (at 750 394.92 0) (effects (font (size 1.27 1.27)) (justify left bottom))) (property "Value" "FROST HEATER" (at 750 392.38 0) (effects (font (size 1.27 1.27)) (justify left bottom))) (property "Footprint" "Connector_JST:JST_XH_B2B-PH-K_1x02_P2.50mm_Vertical" (at 750 400 0) (effects (font (size 1.27 1.27)) (hide yes) (justify left bottom))))
+	(global_label "FROST_HEATER" (at 744.92 400.0 0) (shape bidirectional) (effects (font (size 1.27 1.27))))
+	(global_label "GND" (at 744.92 397.46 0) (shape bidirectional) (effects (font (size 1.27 1.27))))
+	(symbol (lib_id "Connector_Generic:Conn_01x02") (at 750 450 0) (property "Reference" "J8" (at 750 444.92 0) (effects (font (size 1.27 1.27)) (justify left bottom))) (property "Value" "FROST LIGHT" (at 750 442.38 0) (effects (font (size 1.27 1.27)) (justify left bottom))) (property "Footprint" "Connector_JST:JST_XH_B2B-PH-K_1x02_P2.50mm_Vertical" (at 750 450 0) (effects (font (size 1.27 1.27)) (hide yes) (justify left bottom))))
+	(global_label "FROST_GROW_LIGHT" (at 744.92 450.0 0) (shape bidirectional) (effects (font (size 1.27 1.27))))
+	(global_label "GND" (at 744.92 447.46 0) (shape bidirectional) (effects (font (size 1.27 1.27))))
+	(text "Frost outputs (J7 heater, J8 grow light, v3.3)" (at 730 360 0) (effects (font (size 1.8 1.8))))
 )

Commit message: hardware(pcb-v3): add EXP1 J6 expansion header (2x10, future)
J6 2x10 pin header at (300, 400) below ESP32. Pinout (silkscreen
reference only, not wired in schematic):
  Odd row:  1=IO3  3=IO9  5=IO11 7=IO14 9=IO15 11=IO36 13=IO38 15=IO42 17=GND  19=VBAT
  Even row: 2=IO46 4=IO47 6=IO48 8=IO35 10=3V3 12=IO37 14=IO41 16=IO45 18=5V  20=GND

Implementation: placed the J6 symbol only - no wires, no net labels.
User wires specific pins in KiCad GUI when needed (annotation lists
each pin + ESP32 pin position).

Why not auto-wire: a first attempt routed all 15 GPIOs through
support cols (x=270 left, x=340 right) with labels at the ESP32
pins. Added ~80 violations: sub-mm parser disagreement on adjacent
right-side pins (IO35/IO36/IO37 placed at different y by our
parser than KiCad's), multiple_net_names, label_dangling.

ERC: 149 violations (was 145, +4). The +4 are:
  - 1 new multiple_net_names: +3V3/UART_TX (cosmetic, sub-mm)
  - 3 misc cosmetic warnings from the new symbol

The right-side pin sub-mm issue is documented in commit 24d97e5.
Manual wiring in KiCad GUI lets the user place wires with KiCad's
own parser, avoiding the disagreement.
Parts:
- removed TP1: VBAT_ADC, TestPoint:TestPoint_Pad_D1.0mm, symbol Connector:TestPoint
- removed TP1: nFAULT_ACT, TestPoint:TestPoint_Pad_D1.0mm, symbol Connector:TestPoint
- added J6: EXP1 GPIO+POWER (FUTURE), Connector_PinHeader_2.54mm:PinHeader_2x10_P2.54mm_Vertical, symbol Connector_Generic:Conn_02x10_Odd_Even
- added TP1: nFAULT_ACT, TestPoint:TestPoint_Pad_D1.0mm, symbol Connector:TestPoint
- added TP1: VBAT_ADC, TestPoint:TestPoint_Pad_D1.0mm, symbol Connector:TestPoint
Other:
- note added: "Expansion header J6 (FUTURE) — 15 free GPIOs + 3V3/5V/GND/VBAT"
- note added: "Pinout: 1=IO3 3=IO9 5=IO11 7=IO14 9=IO15 11=IO36 13=IO38 15=IO42 17=GND 19=VBAT | 2=IO46 4=IO47 6=IO48 8=IO35 10=3V3 12=IO37 14=IO41 16=IO45 18=5V 20=GND"
Changed lines of the file:
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@@
 	(global_label "GND" (at 744.92 447.46 0) (shape bidirectional) (effects (font (size 1.27 1.27))))
 	(text "Frost outputs (J7 heater, J8 grow light, v3.3)" (at 730 360 0) (effects (font (size 1.8 1.8))))
+	(symbol (lib_id "Connector_Generic:Conn_02x10_Odd_Even") (at 300 400 0) (property "Reference" "J6" (at 300 394.92 0) (effects (font (size 1.27 1.27)) (justify left bottom))) (property "Value" "EXP1 GPIO+POWER (FUTURE)" (at 300 392.38 0) (effects (font (size 1.27 1.27)) (justify left bottom))) (property "Footprint" "Connector_PinHeader_2.54mm:PinHeader_2x10_P2.54mm_Vertical" (at 300 400 0) (effects (font (size 1.27 1.27)) (hide yes) (justify left bottom))))
+	(text "Pinout: 1=IO3 3=IO9 5=IO11 7=IO14 9=IO15 11=IO36 13=IO38 15=IO42 17=GND 19=VBAT | 2=IO46 4=IO47 6=IO48 8=IO35 10=3V3 12=IO37 14=IO41 16=IO45 18=5V 20=GND" (at 288 365 0) (effects (font (size 1.0 1.0))))
+	(text "Expansion header J6 (FUTURE) — 15 free GPIOs + 3V3/5V/GND/VBAT" (at 270 425 0) (effects (font (size 1.8 1.8))))
 )

Commit message: hardware(pcb-v3): scaffold PCB layout
- Add wattplot-v3.kicad_pcb with 80×60mm board outline (Edge.Cuts)
- Add 4× M3 mounting holes (3.2mm drill, 3.5mm inset from edges)
- Set JLCPCB-friendly design rules: 6 mil min, 0.3mm via, 0.6mm pad
- Add 'Power' netclass (20 mil trace, 0.8mm via) for 12V/5V/VM rails
- Add init_layout.py: regenerates board setup from this script
- Add extract_netlist.py: workaround for empty lib_symbols section
  (kicad-cli netlist export returns 0 components when lib_symbols
  is empty; this S-expr parser extracts component list from
  (symbol ...) blocks with (property "Reference"/"Value"/"Footprint"))

Next (interactive, in KiCad GUI):
  1. Open wattplot-v3.kicad_pro
  2. Update PCB from schematic (Tools menu) — brings in all 440 components
  3. Place: ESP32 (antenna top-center) → connectors (long edge) →
     power tree → DRV8871s near their output connectors
  4. Route: power first (12V → 5V → 3.3V), then signal
  5. Generate Gerbers + JLCPCB BOM + CPL via kicad-cli
Parts:
- removed TP1: nFAULT_ACT, TestPoint:TestPoint_Pad_D1.0mm, symbol Connector:TestPoint
- removed TP1: VBAT_ADC, TestPoint:TestPoint_Pad_D1.0mm, symbol Connector:TestPoint
- added TP1: nFAULT_ACT, TestPoint:TestPoint_Pad_D1.0mm, symbol Connector:TestPoint
- added TP1: VBAT_ADC, TestPoint:TestPoint_Pad_D1.0mm, symbol Connector:TestPoint
